File: hardware/diffuino_selector/diffuino_selector.kicad_sch (KiCad schematic)
At the start: 43 parts, among them J1 UNO_Q, Q1 2N3904, SW1 BCD_SELECT, SW2 GENERATE, SW3 RESET, U1 74AHC1G32, U2 74AHC1G08, U3 74AHC1G04, U4 74AHC1G08

Commit message: redraw complete Diffuino selector circuit
Parts:
- removed SW1: BCD_SELECT, Button_Switch_THT:SW_DIP_SPSTx04_Slide_9.78x12.34mm_W7.62mm_P2.54mm, symbol Switch:SW_DIP_x04
- removed SW2: GENERATE, Button_Switch_THT:SW_PUSH_6mm, symbol Switch:SW_Push
- removed SW3: RESET, Button_Switch_THT:SW_PUSH_6mm, symbol Switch:SW_Push
- added SW1: BCD3, Button_Switch_THT:SW_DIP_SPSTx01_Slide_9.78x4.72mm_W7.62mm_P2.54mm, symbol Switch:SW_SPST
- added SW2: BCD2, Button_Switch_THT:SW_DIP_SPSTx01_Slide_9.78x4.72mm_W7.62mm_P2.54mm, symbol Switch:SW_SPST
- added SW3: BCD1, Button_Switch_THT:SW_DIP_SPSTx01_Slide_9.78x4.72mm_W7.62mm_P2.54mm, symbol Switch:SW_SPST
- added SW4: BCD0, Button_Switch_THT:SW_DIP_SPSTx01_Slide_9.78x4.72mm_W7.62mm_P2.54mm, symbol Switch:SW_SPST
- added SW5: GENERATE, Button_Switch_THT:SW_PUSH_6mm, symbol Switch:SW_Push
- added SW6: RESET, Button_Switch_THT:SW_PUSH_6mm, symbol Switch:SW_Push
- D5: value TRIGGER -> GREEN
- J1: value UNO_Q -> ARDUINO_UNO_Q
Connections:
- net B_OR_C is gone; now on an unnamed net: U1.4, U2.2
- net TRIGGER_LED_A is gone; now on net GND: D5.1 (K), R16.2
- net TRIGGER_LED_K is gone; now on net GND: D5.2 (A), Q1.2 (C)
- net +5V: now also C10.1, C11.1, C7.1, C8.1, C9.1, SW1.1 (A), SW2.1 (A), SW3.1 (A), SW4.1 (A), SW5.1, SW6.1; no longer C10.2, C11.2, C7.2, C8.2, C9.2
- net GND: now also C1.2, C10.2, C11.2, C2.2, C3.2, C4.2, C5.2, C6.2, C7.2, C8.2, C9.2, D1.1 (K), D2.1 (K), D3.1 (K), D4.1 (K), R1.2, R13.2, R17.2, R2.2, R3.2, R4.2; no longer C1.1, C10.1, C11.1, C2.1, C3.1, C4.1, C5.1, C6.1, C7.1, C8.1, C9.1, D1.2 (A), D2.2 (A), D3.2 (A), D4.2 (A), R1.1, R13.1, R17.1, R2.1, R3.1, R4.1
- removed net B0R: C4.2, R12.2, R4.2, R8.2
- net B0_D2: no longer names the net of R8.1
- net B0_D2: now also C4.1, R12.1, R4.1, SW4.2 (B); no longer J1.3 (Pin_3)
- removed net B1R: C3.2, R11.2, R3.2, R7.2
- removed net B1_D3: J1.4 (Pin_4), R7.1, U1.2
- removed net B2R: C2.2, R10.2, R2.2, R6.2
- removed net B2_D4: J1.5 (Pin_5), R6.1, U1.1
- removed net B3R: C1.2, R1.2, R5.2, R9.2
- net B3_D5: no longer names the net of J1.6 (Pin_6), U2.1
- net B3_D5: now also R5.2; no longer R5.1
- removed net GENERATE_RAW: C5.2, R13.2, U4.1
- net INVALID: no longer names the net of U2.4, U3.2
- removed net L0A: D4.1 (K), R12.1
- net L1A: no longer names the net of R11.1
- net L1A: now also C3.1, R3.1, R7.1, SW3.2 (B); no longer D3.1 (K)
- net L2A: no longer names the net of R10.1
- net L2A: now also C2.1, R2.1, R6.1, SW2.2 (B); no longer D2.1 (K)
- net L3A: no longer names the net of R9.1
- net L3A: now also C1.1, R1.1, R5.1, SW1.2 (B); no longer D1.1 (K)
- net Q1_BASE: no longer names the net of R15.1
- net Q1_BASE: now also J1.7 (Pin_7), R14.2; no longer Q1.1 (B)
- net RESET_D7: no longer names the net of R18.1
- net RESET_D7: now also C6.1, R17.1, SW6.2; no longer J1.8 (Pin_8)
- removed net RESET_RAW: C6.2, R17.2, R18.2
- removed net TRIGGER: R14.2, R15.2, U4.4
- net TRIG_D6: no longer names the net of R14.1
- net TRIG_D6: now also U4.4; no longer J1.7 (Pin_7)
- net VALID: no longer names the net of U4.2
- net VALID: now also C5.1, R13.1, SW5.2; no longer U3.4
- new net: J1.5 (Pin_5), R6.2, U1.2
- new net: D3.2 (A), R11.2
- new net: J1.8 (Pin_8), R18.2
- new net: U3.4, U4.1
- new net: D1.2 (A), R9.2
- new net: J1.4 (Pin_4), R7.2, U1.1
- new net: J1.3 (Pin_3), R8.2
- new net: D2.2 (A), R10.2
- new net: Q1.1 (B), R15.2
- new net: D4.2 (A), R12.2
Other:
- note added: "1 +5V"
- note added: "1. BCD SELECTOR, INPUT FILTERS, AND VISIBLE BIT INDICATORS"
- note added: "2 GND"
- note added: "2. HARDWARE DECIMAL-VALIDITY INTERLOCK"
- note added: "3 D2 / BCD0"
- note added: "3. DEBOUNCED GENERATE REQUEST"
- note added: "4 D3 / BCD1"
- note added: "4. DEBOUNCED RESET / RE-ARM"
- note added: "5 D4 / BCD2"
- note added: "5. LOCAL SUPPLY DECOUPLING"
- note added: "6 D5 / BCD3"
- note added: "7 D6 / GENERATE"
- note added: "8 D7 / RESET"
- note added: "BCD2 OR BCD1"
- note added: "BCD3 AND previous"
- note added: "BUFFERED REQUEST INDICATOR"
- note added: "D2-D7 are the UNO Q's 5 V-tolerant STM32 header inputs. Never connect this circuit to the 1.8 V MPU GPIO."
- note added: "DIFFUINO — COMPLETE BCD INPUT AND CONTROL CIRCUIT"
- note added: "Firmware: 40 ms debounce; BCD is latched for inference; D6 is ignored while busy; D7 restores the ready smiley."
- note added: "Hardware validity: VALID = NOT [ BCD3 AND (BCD2 OR BCD1) ]"
- note added: "ON = +5 V OFF = 10 kOhm pull-down"
- note added: "U1"
- note added: "U2"
- note added: "U3"
- note added: "U4"
- note added: "UNO Q STM32 HEADER"
- note added: "VALID"
- note removed: "Arduino UNO Q interface"
- note removed: "BCD input and indication"
- note removed: "BCD validity interlock (values 10–15 cannot trigger inference)"
- note removed: "DIFFUINO — 4-BIT BCD SELECTOR, VALIDITY GATE, AND RESET"
- note removed: "Firmware adds 40 ms debounce, ignores D6 while sampling, and latches the result until D7 reset."
- note removed: "Power filtering — place each 100 nF capacitor beside its IC"
- note removed: "Reset / re-arm"
- note removed: "Use only the UNO Q STM32 digital header shown here; do not connect these 5 V nets to 1.8 V MPU GPIO."
- note removed: "VALID = NOT(BCD3 AND (BCD2 OR BCD1)); D6 = GENERATE AND VALID"
- company: (none) -> MonoDiffuse
- title: Diffuino BCD Selector -> Diffuino BCD selector, validity interlock, and reset

Commit message: finalize Diffuino figure and arXiv paper bundle
Connections:
- net GND: no longer D5.1 (K), D5.2 (A), Q1.2 (C), R16.2
- net at J1.6 (Pin_6), R5.2, U2.1: no longer U1.4, U2.2
- new net: D5.1 (K), Q1.2 (C)
- new net: D5.2 (A), R16.2
- new net: U1.4, U2.2
